Commit message: Update ball_handler_robot.urdf

File: ball_handler_robot.urdf (robot description, URDF)
Before this commit: robot my_robot, 10 links, 9 joints
Links:
- removed link gripper
- added link gripper_palm, mass 0.1; collision box size=0.1 0.2 0.05; visual box size=0.1 0.2 0.05
- link gripper_finger_left: mass 0.1 -> 0.05; geometry collision box size=0.1 0.02 0.05; visual box size=0.1 0.02 0.05
- link gripper_finger_right: mass 0.1 -> 0.05; geometry collision box size=0.1 0.02 0.05; visual box size=0.1 0.02 0.05
Joints:
- removed joint gripper_joint
- added joint gripper_palm_joint: type fixed, parent gripper_base, child gripper_palm, origin xyz=0.1 0 0 rpy=0 0 0
- joint front_left_wheel_joint: origin xyz=0.15 0.15 0 rpy=0 0 0 -> xyz=0.15 0.15 -0.05 rpy=0 0 0
- joint front_right_wheel_joint: origin xyz=0.15 -0.15 0 rpy=0 0 0 -> xyz=0.15 -0.15 -0.05 rpy=0 0 0
- joint gripper_base_joint: origin xyz=0.2 0 0.075 rpy=0 0 0 -> xyz=0.25 0 0.075 rpy=0 0 0
- joint gripper_finger_left_joint: axis 1 0 0 -> 0 1 0; limit lower=0 upper=0.1 effort=10 velocity=0.1 -> lower=0 upper=0.05 effort=10 velocity=0.1; origin xyz=-0.1 0 0 rpy=0 0 0 -> xyz=0 0.08 0 rpy=0 0 0; parent gripper -> gripper_palm
- joint gripper_finger_right_joint: axis -1 0 0 -> 0 1 0; limit lower=-0.1 upper=0 effort=10 velocity=0.1 -> lower=-0.05 upper=0 effort=10 velocity=0.1; mimic joint=gripper_finger_left_joint multiplier=-1 -> (none); origin xyz=0.1 0 0 rpy=0 0 0 -> xyz=0 -0.08 0 rpy=0 0 0; parent gripper -> gripper_palm
- joint rear_left_wheel_joint: origin xyz=-0.15 0.15 0 rpy=0 0 0 -> xyz=-0.15 0.15 -0.05 rpy=0 0 0
- joint rear_right_wheel_joint: origin xyz=-0.15 -0.15 0 rpy=0 0 0 -> xyz=-0.15 -0.15 -0.05 rpy=0 0 0
